Commit message: r2000ic210l: update velocities from operators manual

File: fanuc_r2000ic_support/urdf/r2000ic210l_macro.xacro (robot description, xacro)
@@ -122,5 +122,5 @@
       <child link="${prefix}link_2"/>
       <axis xyz="0 1 0"/>
-      <limit lower="${radians(-60)}" upper="${radians(76)}" effort="0" velocity="${radians(90)}"/>
+      <limit lower="${radians(-60)}" upper="${radians(76)}" effort="0" velocity="${radians(85)}"/>
     </joint>
     <joint name="${prefix}joint_3" type="revolute">
