Commit message: limits for J2 and J3 as best case from J2+J3 limits

File: fanuc_m10id_support/urdf/m10id12_macro.xacro (robot description, xacro)
@@ -122,5 +122,5 @@
       <child link="${prefix}link_2"/>
       <axis xyz="0 1 0"/>
-      <limit lower="-1.57" upper="2.79" effort="0" velocity="${radians(240)}"/>
+      <limit lower="${radians(-90)}" upper="${radians(145)}" effort="0" velocity="${radians(240)}"/>
     </joint>
     <joint name="${prefix}joint_3" type="revolute">
@@ -129,5 +129,5 @@
       <child link="${prefix}link_3"/>
       <axis xyz="0 -1 0"/>
-      <limit lower="-3.14" upper="4.61" effort="0" velocity="${radians(260)}"/>
+      <limit lower="${radians(-90)}" upper="${radians(315)}" effort="0" velocity="${radians(260)}"/>
     </joint>
     <joint name="${prefix}joint_4" type="revolute">

Commit message: m-10iD/12 J2,J3,J5,J6 limits from operators manual, for integrated cable type

File: fanuc_m10id_support/urdf/m10id12_macro.xacro (robot description, xacro)
@@ -129,5 +129,5 @@
       <child link="${prefix}link_3"/>
       <axis xyz="0 -1 0"/>
-      <limit lower="${radians(-90)}" upper="${radians(315)}" effort="0" velocity="${radians(260)}"/>
+      <limit lower="${radians(-180)}" upper="${radians(275)}" effort="0" velocity="${radians(260)}"/>
     </joint>
     <joint name="${prefix}joint_4" type="revolute">
@@ -143,5 +143,5 @@
       <child link="${prefix}link_5"/>
       <axis xyz="0 -1 0"/>
-      <limit lower="${radians(-180)}" upper="${radians(180)}" effort="0" velocity="${radians(450)}"/>
+      <limit lower="${radians(-140)}" upper="${radians(140)}" effort="0" velocity="${radians(450)}"/>
     </joint>
     <joint name="${prefix}joint_6" type="revolute">
@@ -150,5 +150,5 @@
       <child link="${prefix}link_6"/>
       <axis xyz="-1 0 0"/>
-      <limit lower="${radians(-450)}" upper="${radians(450)}" effort="0" velocity="${radians(720)}"/>
+      <limit lower="${radians(-270)}" upper="${radians(270)}" effort="0" velocity="${radians(720)}"/>
     </joint>
     <!-- ROS-Industrial 'base' frame: base_link to Fanuc World Coordinates transform -->
