Commit message: M-710/50: limits in degrees

File: fanuc_m710ic_support/urdf/m710ic50_macro.xacro (robot description, xacro)
@@ -115,5 +115,5 @@
       <child link="${prefix}link_1" />
       <axis xyz="0 0 1" />
-      <limit effort="0" lower="-3.1415" upper="3.1415" velocity="3.0543" />
+      <limit effort="0" lower="${radians(-180)}" upper="${radians(180)}" velocity="${radians(175)}" />
     </joint>
     <joint name="${prefix}joint_2" type="revolute">
@@ -122,5 +122,5 @@
       <child link="${prefix}link_2" />
       <axis xyz="0 1 0" />
-      <limit effort="0" lower="-1.5707" upper="2.3561" velocity="3.0543" />
+      <limit effort="0" lower="${radians(-90)}" upper="${radians(135)}" velocity="${radians(175)}" />
     </joint>
     <joint name="${prefix}joint_3" type="revolute">
@@ -129,5 +129,5 @@
       <child link="${prefix}link_3" />
       <axis xyz="0 -1 0" />
-      <limit effort="0" lower="-2.7925" upper="4.8869" velocity="3.0543" />
+      <limit effort="0" lower="${radians(-160)}" upper="${radians(280)}" velocity="${radians(175)}" />
     </joint>
     <joint name="${prefix}joint_4" type="revolute">
@@ -136,5 +136,5 @@
       <child link="${prefix}link_4"/>
       <axis xyz="-1 0 0"/>
-      <limit effort="0" lower="-6.2830" upper="6.2830" velocity="4.3633" />
+      <limit effort="0" lower="${radians(-360)}" upper="${radians(360)}" velocity="${radians(250)}" />
     </joint>
     <joint name="${prefix}joint_5" type="revolute">
@@ -143,5 +143,5 @@
       <child link="${prefix}link_5"/>
       <axis xyz="0 -1 0"/>
-      <limit effort="0" lower="-2.1816" upper="2.1816" velocity="4.3633" />
+      <limit effort="0" lower="${radians(-125)}" upper="${radians(125)}" velocity="${radians(250)}" />
     </joint>
     <joint name="${prefix}joint_6" type="revolute">
@@ -150,5 +150,5 @@
       <child link="${prefix}link_6"/>
       <axis xyz="-1 0 0"/>
-      <limit effort="0" lower="-6.2831" upper="6.2831" velocity="6.1959" />
+      <limit effort="0" lower="${radians(-360)}" upper="${radians(360)}" velocity="${radians(355)}" />
     </joint>
     <!-- ROS-Industrial 'base' frame: base_link to Fanuc World Coordinates transform -->
