Commit message: Fix axis limits for crx10ia A1 and A6  and crx10ial A6

File: fanuc_crx10ia_support/urdf/crx10ia_macro.xacro (robot description, xacro)
@@ -115,5 +115,5 @@
       <child link="${prefix}link_1" />
       <axis xyz="0 0 1" />
-      <limit effort="0" lower="${radians(-180)}" upper="${radians(180)}" velocity="${radians(120)}" />
+      <limit effort="0" lower="${radians(-190)}" upper="${radians(190)}" velocity="${radians(120)}" />
     </joint>
     <joint name="${prefix}joint_2" type="revolute">
@@ -150,5 +150,5 @@
       <child link="${prefix}link_6"/>
       <axis xyz="-1 0 0"/>
-      <limit effort="0" lower="${radians(-190)}" upper="${radians(190)}" velocity="${radians(180)}" />
+      <limit effort="0" lower="${radians(-225)}" upper="${radians(225)}" velocity="${radians(180)}" />
     </joint>
     <!-- ROS-Industrial 'base' frame: base_link to Fanuc World Coordinates transform -->

File: fanuc_crx10ia_support/urdf/crx10ial_macro.xacro (robot description, xacro)
@@ -150,5 +150,5 @@
       <child link="${prefix}link_6"/>
       <axis xyz="-1 0 0"/>
-      <limit effort="0" lower="${radians(-190)}" upper="${radians(190)}" velocity="${radians(180)}" />
+      <limit effort="0" lower="${radians(-225)}" upper="${radians(225)}" velocity="${radians(180)}" />
     </joint>
     <!-- ROS-Industrial 'base' frame: base_link to Fanuc World Coordinates transform -->
