Commit message: fix motion limits based on Operators Manual

File: fanuc_m20id_support/urdf/m20id25_macro.xacro (robot description, xacro)
@@ -115,5 +115,5 @@
       <child link="${prefix}link_1"/>
       <axis xyz="0 0 1"/>
-      <limit lower="${radians(-340)}" upper="${radians(340)}" effort="0" velocity="${radians(210)}" />
+      <limit lower="${radians(-170)}" upper="${radians(170)}" effort="0" velocity="${radians(210)}" />
     </joint>
     <joint name="${prefix}joint_2" type="revolute">
@@ -122,5 +122,5 @@
       <child link="${prefix}link_2"/>
       <axis xyz="0 1 0"/>
-      <limit lower="${radians(-260)}" upper="${radians(260)}" effort="0" velocity="${radians(210)}" />
+      <limit lower="${radians(-100)}" upper="${radians(160)}" effort="0" velocity="${radians(210)}" />
     </joint>
     <joint name="${prefix}joint_3" type="revolute">
@@ -129,5 +129,5 @@
       <child link="${prefix}link_3"/>
       <axis xyz="0 -1 0"/>
-      <limit lower="${radians(-458)}" upper="${radians(458)}" effort="0" velocity="${radians(265)}" />
+      <limit lower="${radians(-190)}" upper="${radians(268)}" effort="0" velocity="${radians(265)}" />
     </joint>
     <joint name="${prefix}joint_4" type="revolute">
@@ -136,5 +136,5 @@
       <child link="${prefix}link_4"/>
       <axis xyz="0 0 -1"/>
-      <limit lower="${radians(-400)}" upper="${radians(400)}" effort="0" velocity="${radians(420)}" />
+      <limit lower="${radians(-200)}" upper="${radians(200)}" effort="0" velocity="${radians(420)}" />
     </joint>
     <joint name="${prefix}joint_5" type="revolute">
@@ -143,5 +143,5 @@
       <child link="${prefix}link_5"/>
       <axis xyz="0 -1 0"/>
-      <limit lower="${radians(-280)}" upper="${radians(280)}" effort="0" velocity="${radians(420)}" />
+      <limit lower="${radians(-140)}" upper="${radians(140)}" effort="0" velocity="${radians(420)}" />
     </joint>
     <joint name="${prefix}joint_6" type="revolute">
@@ -150,5 +150,5 @@
       <child link="${prefix}link_6"/>
       <axis xyz="0 0 -1"/>
-      <limit lower="${radians(-540)}" upper="${radians(540)}" effort="0" velocity="${radians(720)}" />
+      <limit lower="${radians(-270)}" upper="${radians(270)}" effort="0" velocity="${radians(720)}" />
     </joint>
     <!-- ROS-Industrial 'base' frame: base_link to Fanuc World Coordinates transform -->

Commit message: m20id25: fix j3 limits, remove unused mesh

File: fanuc_m20id_support/urdf/m20id25_macro.xacro (robot description, xacro)
@@ -129,5 +129,5 @@
       <child link="${prefix}link_3"/>
       <axis xyz="0 -1 0"/>
-      <limit lower="${radians(-190)}" upper="${radians(268)}" effort="0" velocity="${radians(265)}" />
+      <limit lower="${radians(-190)}" upper="${radians(268.4)}" effort="0" velocity="${radians(265)}" />
     </joint>
     <joint name="${prefix}joint_4" type="revolute">

Commit message: mixed version, other urdf and meshes by alpkocabas

File: fanuc_m20id_support/urdf/m20id25_macro.xacro (robot description, xacro)
@@ -1,25 +1,30 @@
-<?xml version="1.0"?>
+<?xml version="1.0" encoding="utf-8"?>
 <robot xmlns:xacro="http://wiki.ros.org/xacro">
   <xacro:include filename="$(find fanuc_resources)/urdf/common_materials.xacro"/>
   <xacro:macro name="fanuc_m20id25" params="prefix">
-    <!-- links: main serial chain -->
     <link name="${prefix}base_link">
-      <visual>
-        <origin xyz="0 0 0" rpy="0 0 0"/>
-        <geometry>
-          <mesh filename="package://fanuc_m20id_support/meshes/m20id25/visual/base_link.stl"/>
-        </geometry>
-        <xacro:material_fanuc_gray28 />
-      </visual>
-      <collision>
-        <origin xyz="0 0 0" rpy="0 0 0"/>
-        <geometry>
-          <mesh filename="package://fanuc_m20id_support/meshes/m20id25/collision/base_link.stl"/>
-        </geometry>
-      </collision>
+    <visual>
+      <origin
+        xyz="0 0 0"
+        rpy="0 0 0" />
+      <geometry>
+        <mesh filename="package://fanuc_m20id_support/meshes/m20id25/visual/base_link.stl"/>
+      </geometry>
+      <xacro:material_fanuc_gray28 />
+    </visual>
+    <collision>
+      <origin
+        xyz="0 0 0"
+        rpy="0 0 0" />
+      <geometry>
+        <mesh filename="package://fanuc_m20id_support/meshes/m20id25/collision/base_link.stl"/>
+      </geometry>
+    </collision>
     </link>
     <link name="${prefix}link_1">
       <visual>
-        <origin xyz="0 0 0" rpy="0 0 0"/>
+        <origin
+          xyz="0 0 0"
+          rpy="0 0 0" />
         <geometry>
           <mesh filename="package://fanuc_m20id_support/meshes/m20id25/visual/link_1.stl"/>
@@ -28,5 +33,7 @@
       </visual>
       <collision>
-        <origin xyz="0 0 0" rpy="0 0 0"/>
+        <origin
+          xyz="0 0 0"
+          rpy="0 0 0" />
         <geometry>
           <mesh filename="package://fanuc_m20id_support/meshes/m20id25/collision/link_1.stl"/>
@@ -36,5 +43,7 @@
     <link name="${prefix}link_2">
       <visual>
-        <origin xyz="0 0 0" rpy="0 0 0"/>
+        <origin
+          xyz="0 0 0"
+          rpy="0 0 0" />
         <geometry>
           <mesh filename="package://fanuc_m20id_support/meshes/m20id25/visual/link_2.stl"/>
@@ -42,114 +51,89 @@
         <xacro:material_fanuc_yellow />
       </visual>
-      <collision>
-        <origin xyz="0 0 0" rpy="0 0 0"/>
-        <geometry>
-          <mesh filename="package://fanuc_m20id_support/meshes/m20id25/collision/link_2.stl"/>
-        </geometry>
-      </collision>
+    <collision>
+      <origin
+        xyz="0 0 0"
+        rpy="0 0 0" />
+      <geometry>
+        <mesh filename="package://fanuc_m20id_support/meshes/m20id25/visual/link_2.stl"/>
+      </geometry>
+    </collision>
     </link>
     <link name="${prefix}link_3">
-      <visual>
-        <origin xyz="0 0 0" rpy="0 0 0"/>
-        <geometry>
-          <mesh filename="package://fanuc_m20id_support/meshes/m20id25/visual/link_3.stl"/>
-        </geometry>
-        <xacro:material_fanuc_yellow />
-      </visual>
-      <collision>
-        <origin xyz="0 0 0" rpy="0 0 0"/>
-        <geometry>
-          <mesh filename="package://fanuc_m20id_support/meshes/m20id25/collision/link_3.stl"/>
-        </geometry>
-      </collision>
+    <visual>
+      <origin
+        xyz="0 0 0"
+        rpy="0 0 0" />
+      <geometry>
+        <mesh filename="package://fanuc_m20id_support/meshes/m20id25/visual/link_3.stl"/>
+      </geometry>
+      <xacro:material_fanuc_yellow />
+    </visual>
+    <collision>
+      <origin
+        xyz="0 0 0"
+        rpy="0 0 0" />
+      <geometry>
+        <mesh filename="package://fanuc_m20id_support/meshes/m20id25/collision/link_3.stl"/>
+      </geometry>
+    </collision>
     </link>
     <link name="${prefix}link_4">
-      <visual>
-        <origin xyz="0 0 0" rpy="0 0 0"/>
-        <geometry>
-          <mesh filename="package://fanuc_m20id_support/meshes/m20id25/visual/link_4.stl"/>
-        </geometry>
-        <xacro:material_fanuc_yellow />
-      </visual>
-      <collision>
-        <origin xyz="0 0 0" rpy="0 0 0"/>
-        <geometry>
-          <mesh filename="package://fanuc_m20id_support/meshes/m20id25/collision/link_4.stl"/>
-        </geometry>
-      </collision>
+    <visual>
+      <origin
+        xyz="0 0 0"
+        rpy="0 0 0" />
+      <geometry>
+        <mesh filename="package://fanuc_m20id_support/meshes/m20id25/visual/link_4.stl"/>
+      </geometry>
+      <xacro:material_fanuc_yellow />
+    </visual>
+    <collision>
+      <origin
+        xyz="0 0 0"
+        rpy="0 0 0" />
+      <geometry>
+        <mesh filename="package://fanuc_m20id_support/meshes/m20id25/collision/link_4.stl"/>
+      </geometry>
+    </collision>
     </link>
     <link name="${prefix}link_5">
-      <visual>
-        <origin xyz="0 0 0" rpy="0 0 0"/>
-        <geometry>
-          <mesh filename="package://fanuc_m20id_support/meshes/m20id25/visual/link_5.stl"/>
-        </geometry>
-        <xacro:material_fanuc_yellow />
-      </visual>
-      <collision>
-        <origin xyz="0 0 0" rpy="0 0 0"/>
-        <geometry>
-          <mesh filename="package://fanuc_m20id_support/meshes/m20id25/collision/link_5.stl"/>
-        </geometry>
-      </collision>
+    <visual>
+      <origin
+        xyz="0 0 0"
+        rpy="0 0 0" />
+      <geometry>
+        <mesh filename="package://fanuc_m20id_support/meshes/m20id25/visual/link_5.stl"/>
+      </geometry>
+      <xacro:material_fanuc_yellow />
+    </visual>
+    <collision>
+      <origin
+        xyz="0 0 0"
+        rpy="0 0 0" />
+      <geometry>
+        <mesh filename="package://fanuc_m20id_support/meshes/m20id25/collision/link_5.stl"/>
+      </geometry>
+    </collision>
     </link>
     <link name="${prefix}link_6">
-      <visual>
-        <origin xyz="0 0 0" rpy="0 0 0"/>
-        <geometry>
-          <mesh filename="package://fanuc_m20id_support/meshes/m20id25/visual/link_6.stl"/>
-        </geometry>
-        <xacro:material_fanuc_black />
-      </visual>
-      <collision>
-        <origin xyz="0 0 0" rpy="0 0 0"/>
-        <geometry>
-          <mesh filename="package://fanuc_m20id_support/meshes/m20id25/collision/link_6.stl"/>
-        </geometry>
-      </collision>
-    </link>
-    <!-- joints: main serial chain -->
-    <joint name="${prefix}joint_1" type="revolute">
-      <origin xyz="0 0 0.425" rpy="0 0 0"/>
-      <parent link="${prefix}base_link"/>
-      <child link="${prefix}link_1"/>
-      <axis xyz="0 0 1"/>
-      <limit lower="${radians(-170)}" upper="${radians(170)}" effort="0" velocity="${radians(210)}" />
-    </joint>
-    <joint name="${prefix}joint_2" type="revolute">
-      <origin xyz="0.075 0 0" rpy="0 0 0"/>
-      <parent link="${prefix}link_1"/>
-      <child link="${prefix}link_2"/>
-      <axis xyz="0 1 0"/>
-      <limit lower="${radians(-100)}" upper="${radians(160)}" effort="0" velocity="${radians(210)}" />
-    </joint>
-    <joint name="${prefix}joint_3" type="revolute">
-      <origin xyz="0 0 0.840" rpy="0 ${radians(90)} 0"/>
-      <parent link="${prefix}link_2"/>
-      <child link="${prefix}link_3"/>
-      <axis xyz="0 -1 0"/>
-      <limit lower="${radians(-190)}" upper="${radians(268.4)}" effort="0" velocity="${radians(265)}" />
-    </joint>
-    <joint name="${prefix}joint_4" type="revolute">
-      <origin xyz="-0.215 0 0.890" rpy="0 0 0"/>
-      <parent link="${prefix}link_3"/>
-      <child link="${prefix}link_4"/>
-      <axis xyz="0 0 -1"/>
-      <limit lower="${radians(-200)}" upper="${radians(200)}" effort="0" velocity="${radians(420)}" />
-    </joint>
-    <joint name="${prefix}joint_5" type="revolute">
-      <origin xyz="0 0 0" rpy="0 0 0"/>
-      <parent link="${prefix}link_4"/>
-      <child link="${prefix}link_5"/>
-      <axis xyz="0 -1 0"/>
-      <limit lower="${radians(-140)}" upper="${radians(140)}" effort="0" velocity="${radians(420)}" />
-    </joint>
-    <joint name="${prefix}joint_6" type="revolute">
-      <origin xyz="0 0 0.09" rpy="0 0 0"/>
-      <parent link="${prefix}link_5"/>
-      <child link="${prefix}link_6"/>
-      <axis xyz="0 0 -1"/>
-      <limit lower="${radians(-270)}" upper="${radians(270)}" effort="0" velocity="${radians(720)}" />
-    </joint>
+    <visual>
+      <origin
+        xyz="0 0 0"
+        rpy="0 0 0" />
+      <geometry>
+        <mesh filename="package://fanuc_m20id_support/meshes/m20id25/visual/link_6.stl"/>
+      </geometry>
+      <xacro:material_fanuc_yellow />
+    </visual>
+    <collision>
+      <origin
+        xyz="0 0 0"
+        rpy="0 0 0" />
+      <geometry>
+        <mesh filename="package://fanuc_m20id_support/meshes/m20id25/collision/link_6.stl"/>
+      </geometry>
+    </collision>
+    </link>
     <!-- ROS-Industrial 'base' frame: base_link to Fanuc World Coordinates transform -->
     <link name="${prefix}base" />
@@ -159,4 +143,64 @@
       <child link="${prefix}base"/>
     </joint>
+    <joint name="${prefix}joint_1" type="revolute">
+      <origin
+        xyz="0 0 0.425"
+        rpy="0 0 0.0" />
+      <parent link="${prefix}base_link"/>
+      <child link="${prefix}link_1"/>
+      <axis
+        xyz="0 0 1" />
+      <limit lower="${radians(-185)}" upper="${radians(185)}" effort="0" velocity="${radians(210)}" />
+    </joint>
+    <joint name="${prefix}joint_2" type="revolute">
+      <origin
+        xyz="0.075 0 0"
+        rpy="0 0 0" />
+      <parent link="${prefix}link_1"/>
+      <child link="${prefix}link_2"/>
+      <axis
+        xyz="0 1 0" />
+      <limit lower="${radians(-100)}" upper="${radians(160)}" effort="0" velocity="${radians(210)}" />
+    </joint>
+    <joint name="${prefix}joint_3" type="revolute">
+      <origin
+        xyz="0 0 0.84"
+        rpy="0 0 0" />
+      <parent link="${prefix}link_2"/>
+      <child link="${prefix}link_3"/>
+      <axis
+        xyz="0 -1 0" />
+      <limit lower="${radians(-190)}" upper="${radians(268)}" effort="0" velocity="${radians(265)}" />
+    </joint>
+    <joint name="${prefix}joint_4" type="revolute">
+      <origin
+        xyz="0 0 0.215"
+        rpy="0 0 0" />
+      <parent link="${prefix}link_3"/>
+      <child link="${prefix}link_4"/>
+      <axis
+        xyz="-1 0 0" />
+      <limit lower="${radians(-200)}" upper="${radians(200)}" effort="0" velocity="${radians(420)}" />
+    </joint>
+    <joint name="${prefix}joint_5" type="revolute">
+      <origin
+        xyz="0.89 0 0"
+        rpy="0 0 0" />
+      <parent link="${prefix}link_4"/>
+      <child link="${prefix}link_5"/>
+      <axis
+        xyz="0 -1 0" />
+      <limit lower="${radians(-180)}" upper="${radians(180)}" effort="0" velocity="${radians(420)}" />
+    </joint>
+    <joint name="${prefix}joint_6" type="revolute">
+      <origin
+        xyz="0.09 0 0"
+        rpy="0 0 0" />
+      <parent link="${prefix}link_5"/>
+      <child link="${prefix}link_6"/>
+      <axis
+        xyz="-1 0 0" />
+      <limit lower="${radians(-270)}" upper="${radians(270)}" effort="0" velocity="${radians(880)}" />
+    </joint>
     <!-- ROS-Industrial 'flange' frame: attachment point for EEF models -->
     <link name="${prefix}flange" />
@@ -169,5 +213,5 @@
     <link name="${prefix}tool0" />
     <joint name="${prefix}link_6-tool0" type="fixed">
-      <origin xyz="0 0 0" rpy="0 0 0" />
+      <origin xyz="0 0 0" rpy="${pi} ${-pi/2.0} 0" />
       <parent link="${prefix}flange" />
       <child link="${prefix}tool0" />
